File: LED_Module/LED_Module.kicad_pcb (KiCad board)
At the start: 2 copper layers, 67.3 x 31.1 mm, 31 parts, among them J1 INPUT, J2 BUS, J3 POWER_REG, Q1 PZT2222A, Q2 PZT2222A, Q3 PZT2222A, Q4 PZT2222A

Commit message: Adding NEMA0183
Parts:
- removed ? (x2), REF** (x2): 1pin, Connectors:1pin
- removed D1: D_BAT, Diodes_THT:D_DO-41_SOD81_P7.62mm_Horizontal
- removed D2: D_BUS, Diodes_THT:D_DO-41_SOD81_P7.62mm_Horizontal
- removed D3, D4, D5, D6: L130-40, LEDs:LED_1206_HandSoldering
- removed D7: LED RED, LEDs:LED_D3.0mm
- removed D8: LED GREEN, LEDs:LED_D3.0mm
- removed D9: LED BLUE, LEDs:LED_D3.0mm
- removed J1: INPUT, Pin_Headers:Pin_Header_Straight_2x04_Pitch2.54mm
- removed J2: BUS, Pin_Headers:Pin_Header_Straight_1x05_Pitch2.54mm
- removed J3: POWER_REG, Pin_Headers:Pin_Header_Straight_1x04_Pitch2.54mm
- removed Q1, Q2, Q3, Q4: PZT2222A, digikey-footprints:SOT-223
- removed R1, R2, R3, R4: 470, Resistors_SMD:R_1206_HandSoldering
- removed R10, R9: 10, Resistors_SMD:R_1206_HandSoldering
- removed R11, R5, R6, R7, R8: 6.8, Resistors_SMD:R_1206_HandSoldering
Routing:
- net GND: track 96.5 -> 0.00 mm
- net Net-(D3-Pad1): track 88.6 -> 0.00 mm
- net Net-(J2-Pad5): track 69.9 -> 0.00 mm
- net Net-(Q1-Pad1): track 40.2 -> 0.00 mm
- net Net-(Q2-Pad1): track 30.8 -> 0.00 mm
- net Net-(D1-Pad1): track 26.5 -> 0.00 mm
- net Net-(Q3-Pad1): track 22.4 -> 0.00 mm
- net Net-(D7-Pad1): track 17.1 -> 0.00 mm
- net Net-(Q4-Pad1): track 13.1 -> 0.00 mm
- net Net-(D8-Pad1): track 11.8 -> 0.00 mm
- net Net-(D2-Pad2): track 10.5 -> 0.00 mm
- net Net-(D9-Pad1): track 9.67 -> 0.00 mm
- net Net-(D6-Pad2): track 7.75 -> 0.00 mm
- net Net-(D3-Pad2): track 7.75 -> 0.00 mm
- net Net-(D5-Pad2): track 5.17 -> 0.00 mm
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Other:
- board outline removed
- net class Default: via_dia 0.6 -> 0.8
- board text removed: "3.3"
- board text removed: "B"
- board text removed: "BAT"
- board text removed: "BUS"
- board text removed: "G"
- board text removed: "GND"
- board text removed: "IN"
- board text removed: "NC"
- board text removed: "R"
- board text removed: "W"
