File: LED_Module/LED_Module.sch (KiCad schematic (older format))
At the start: 27 parts, among them J1 INPUT, J2 BUS, J3 POWER_REG, Q1 PZT2222A, Q2 PZT2222A, Q3 PZT2222A, Q4 PZT2222A

Commit message: Adding NEMA0183
Parts:
- D1, D2: footprint Diodes_THT:D_DO-41_SOD81_P7.62mm_Horizontal -> Diode_THT:D_DO-41_SOD81_P7.62mm_Horizontal; symbol D_Schottky -> LED_Module-rescue:D_Schottky-device
- D3, D4, D5, D6: footprint LEDs:LED_1206_HandSoldering -> LED_SMD:LED_1206_3216Metric_Pad1.42x1.75mm_HandSolder; symbol LED -> LED_Module-rescue:LED-device
- D7, D8, D9: footprint LEDs:LED_D3.0mm -> LED_THT:LED_D3.0mm; symbol LED -> LED_Module-rescue:LED-device
- J1: footprint Pin_Headers:Pin_Header_Straight_2x04_Pitch2.54mm -> Connector_PinHeader_2.54mm:PinHeader_2x04_P2.54mm_Vertical; symbol Conn_02x04_Odd_Even -> LED_Module-rescue:Conn_02x04_Odd_Even-LED_Module-rescue
- J2: footprint Pin_Headers:Pin_Header_Straight_1x05_Pitch2.54mm -> Connector_PinHeader_2.54mm:PinHeader_1x05_P2.54mm_Vertical; symbol Conn_01x05 -> LED_Module-rescue:Conn_01x05-LED_Module-rescue
- J3: footprint Pin_Headers:Pin_Header_Straight_1x04_Pitch2.54mm -> Connector_PinHeader_2.54mm:PinHeader_1x04_P2.54mm_Vertical; symbol Conn_01x04 -> LED_Module-rescue:Conn_01x04-LED_Module-rescue
- Q1, Q2, Q3, Q4: footprint digikey-footprints:SOT-223 -> Package_TO_SOT_SMD:SOT-223-3_TabPin2; symbol Q_NPN_BCEC -> LED_Module-rescue:Q_NPN_BCEC-device
- R1, R10, R11, R2, R3, R4, R5, R6, R7, R8, R9: footprint Resistors_SMD:R_1206_HandSoldering -> Resistor_SMD:R_1206_3216Metric_Pad1.42x1.75mm_HandSolder; symbol R -> LED_Module-rescue:R-device
