File: USB_Power_Filter/USB_Power_Filter.sch (KiCad schematic (older format))
At the start: 13 parts, among them SW1 SW_SPDT, U1 LD1117S33TR_SOT223

Commit message: Adding NEMA0183
Parts:
- removed C4: 100nF, Capacitors_SMD:C_1206_HandSoldering, symbol Device:C
- removed D2: 1N4001, Diode_THT:D_DO-41_SOD81_P10.16mm_Horizontal, symbol Diode:1N4001
- removed SW1: SW_SPDT, symbol Switch:SW_SPDT
- added C2: 1uF, Capacitor_SMD:C_0805_2012Metric_Pad1.15x1.40mm_HandSolder, symbol Device:C
- C1: value 220uF -> UCL1E100MCL; footprint Capacitors_SMD:CP_Elec_6.3x5.8 -> Capacitor_SMD:CP_Elec_4x5.8
- C3: renamed from C2; footprint Capacitors_SMD:C_1206_HandSoldering -> Capacitor_SMD:C_0805_2012Metric_Pad1.15x1.40mm_HandSolder
- C4: renamed from C3; footprint Capacitors_SMD:C_1206_HandSoldering -> Capacitor_SMD:C_0805_2012Metric_Pad1.15x1.40mm_HandSolder
- C5: value 10uF -> 4.7uF; footprint Capacitors_SMD:C_1206_HandSoldering -> Capacitor_SMD:C_0805_2012Metric_Pad1.15x1.40mm_HandSolder
- D1: footprint Diodes_SMD:D_SMB_Handsoldering -> Diode_SMD:D_SMB_Handsoldering
- POWER1: footprint Pin_Headers:Pin_Header_Straight_1x02_Pitch2.54mm -> Connector_PinHeader_2.54mm:PinHeader_1x02_P2.54mm_Vertical
- POWER_IN1: footprint Pin_Headers:Pin_Header_Straight_1x02_Pitch2.54mm -> Connector_Wire:SolderWirePad_1x02_P3.81mm_Drill1mm
- SHIELD1: footprint (none) -> Connector_Wire:SolderWirePad_1x01_Drill1mm
- U1: value LD1117S33TR_SOT223 -> LDL1117S
- USB1: value USB_B_Micro -> Wuerth_629105150521; footprint Connectors_USB:USB_Micro-B_Molex-105017-0001 -> Connector_USB:USB_Micro-B_Wuerth_629105150521_CircularHoles
Connections:
- wire segments 35 -> 27
Other:
- moved on the sheet: C3, C4, C5, POWER1, U1
Changed lines of the file:
@@
 EESchema Schematic File Version 4
-LIBS:USB_Power_Filter-cache
 EELAYER 26 0
 EELAYER END
@@
 U 1 1 5B5E11CC
 P 5700 3600
-F 0 "C1" H 5818 3646 50  0000 L CNN
-F 1 "220uF" H 5818 3555 50  0000 L CNN
-F 2 "Capacitors_SMD:CP_Elec_6.3x5.8" H 5738 3450 50  0001 C CNN
+F 0 "C1" H 5650 3250 50  0000 L CNN
+F 1 "UCL1E100MCL" H 5400 3350 50  0000 L CNN
+F 2 "Capacitor_SMD:CP_Elec_4x5.8" H 5738 3450 50  0001 C CNN
 F 3 "~" H 5700 3600 50  0001 C CNN
 	1    5700 3600
@@
 $EndComp
 $Comp
-L Device:C C2
+L Device:C C3
 U 1 1 5B5E1202
-P 6050 3600
-F 0 "C2" H 6165 3646 50  0000 L CNN
-F 1 "100nF" H 6165 3555 50  0000 L CNN
-F 2 "Capacitors_SMD:C_1206_HandSoldering" H 6088 3450 50  0001 C CNN
-F 3 "~" H 6050 3600 50  0001 C CNN
-	1    6050 3600
-	1    0    0    -1
-$EndComp
-$Comp
-L Device:C C3
-U 1 1 5B5E124E
 P 6400 3600
 F 0 "C3" H 6515 3646 50  0000 L CNN
-F 1 "1nF" H 6515 3555 50  0000 L CNN
-F 2 "Capacitors_SMD:C_1206_HandSoldering" H 6438 3450 50  0001 C CNN
+F 1 "100nF" H 6515 3555 50  0000 L CNN
+F 2 "Capacitor_SMD:C_0805_2012Metric_Pad1.15x1.40mm_HandSolder" H 6438 3450 50  0001 C CNN
 F 3 "~" H 6400 3600 50  0001 C CNN
 	1    6400 3600
+	1    0    0    -1
+$EndComp
+$Comp
+L Device:C C4
+U 1 1 5B5E124E
+P 6750 3600
+F 0 "C4" H 6865 3646 50  0000 L CNN
+F 1 "1nF" H 6865 3555 50  0000 L CNN
+F 2 "Capacitor_SMD:C_0805_2012Metric_Pad1.15x1.40mm_HandSolder" H 6788 3450 50  0001 C CNN
+F 3 "~" H 6750 3600 50  0001 C CNN
+	1    6750 3600
 	1    0    0    -1
 $EndComp
@@
 F 0 "D1" V 5304 3679 50  0000 L CNN
 F 1 "D_TVS" V 5395 3679 50  0000 L CNN
-F 2 "Diodes_SMD:D_SMB_Handsoldering" H 5350 3600 50  0001 C CNN
+F 2 "Diode_SMD:D_SMB_Handsoldering" H 5350 3600 50  0001 C CNN
 F 3 "~" H 5350 3600 50  0001 C CNN
 	1    5350 3600
@@
 L Connector:Conn_01x02_Female POWER1
 U 1 1 5B5E164D
-P 8300 4200
-F 0 "POWER1" V 8200 3700 50  0000 L CNN
-F 1 "Conn_01x02_Female" V 8300 3250 50  0000 L CNN
-F 2 "Pin_Headers:Pin_Header_Straight_1x02_Pitch2.54mm" H 8300 4200 50  0001 C CNN
-F 3 "~" H 8300 4200 50  0001 C CNN
-	1    8300 4200
+P 7750 4000
+F 0 "POWER1" V 7650 3500 50  0000 L CNN
+F 1 "Conn_01x02_Female" V 7750 3050 50  0000 L CNN
+F 2 "Connector_PinHeader_2.54mm:PinHeader_1x02_P2.54mm_Vertical" H 7750 4000 50  0001 C CNN
+F 3 "~" H 7750 4000 50  0001 C CNN
+	1    7750 4000
 	0    1    1    0
 $EndComp
@@
 P 4700 3650
 F 0 "USB1" H 4755 4117 50  0000 C CNN
-F 1 "USB_B_Micro" H 4755 4026 50  0000 C CNN
-F 2 "Connectors_USB:USB_Micro-B_Molex-105017-0001" H 4850 3600 50  0001 C CNN
+F 1 "Wuerth_629105150521" H 4755 4026 50  0000 C CNN
+F 2 "Connector_USB:USB_Micro-B_Wuerth_629105150521_CircularHoles" H 4850 3600 50  0001 C CNN
 F 3 "~" H 4850 3600 50  0001 C CNN
 	1    4700 3650
@@
 F 0 "POWER_IN1" V 5400 3100 50  0000 C CNN
 F 1 "Conn_01x02_Female" V 5300 3100 50  0000 C CNN
-F 2 "Pin_Headers:Pin_Header_Straight_1x02_Pitch2.54mm" H 5250 3100 50  0001 C CNN
+F 2 "Connector_Wire:SolderWirePad_1x02_P3.81mm_Drill1mm" H 5250 3100 50  0001 C CNN
 F 3 "~" H 5250 3100 50  0001 C CNN
 	1    5250 3100
@@
 L Regulator_Linear:LD1117S33TR_SOT223 U1
 U 1 1 5B60B014
-P 7550 3350
-F 0 "U1" H 7550 3592 50  0000 C CNN
-F 1 "LD1117S33TR_SOT223" H 7550 3501 50  0000 C CNN
-F 2 "Package_TO_SOT_SMD:SOT-223-3_TabPin2" H 7550 3550 50  0001 C CNN
-F 3 "http://www.st.com/st-web-ui/static/active/en/resource/technical/document/datasheet/CD00000544.pdf" H 7650 3100 50  0001 C CNN
-	1    7550 3350
+P 7150 3450
+F 0 "U1" H 7150 3692 50  0000 C CNN
+F 1 "LDL1117S" H 7150 3601 50  0000 C CNN
+F 2 "Package_TO_SOT_SMD:SOT-223-3_TabPin2" H 7150 3650 50  0001 C CNN
+F 3 "http://www.st.com/st-web-ui/static/active/en/resource/technical/document/datasheet/CD00000544.pdf" H 7250 3200 50  0001 C CNN
+	1    7150 3450
 	1    0    0    -1
 $EndComp
@@
 L Device:C C5
 U 1 1 5B60C803
-P 7950 3600
-F 0 "C5" H 8065 3646 50  0000 L CNN
-F 1 "10uF" H 8065 3555 50  0000 L CNN
-F 2 "Capacitors_SMD:C_1206_HandSoldering" H 7988 3450 50  0001 C CNN
-F 3 "~" H 7950 3600 50  0001 C CNN
-	1    7950 3600
-	1    0    0    -1
-$EndComp
-$Comp
-L Device:C C4
-U 1 1 5B6164C7
-P 7150 3600
-F 0 "C4" H 7265 3646 50  0000 L CNN
-F 1 "100nF" H 7265 3555 50  0000 L CNN
-F 2 "Capacitors_SMD:C_1206_HandSoldering" H 7188 3450 50  0001 C CNN
-F 3 "~" H 7150 3600 50  0001 C CNN
-	1    7150 3600
+P 7550 3600
+F 0 "C5" H 7665 3646 50  0000 L CNN
+F 1 "4.7uF" H 7665 3555 50  0000 L CNN
+F 2 "Capacitor_SMD:C_0805_2012Metric_Pad1.15x1.40mm_HandSolder" H 7588 3450 50  0001 C CNN
+F 3 "~" H 7550 3600 50  0001 C CNN
+	1    7550 3600
 	1    0    0    -1
 $EndComp
@@
 Connection ~ 5150 3750
 Wire Wire Line
-	5150 3750 5350 3750
-$Comp
-L Switch:SW_SPDT SW1
-U 1 1 5B620940
-P 6800 3450
-F 0 "SW1" H 6800 3735 50  0000 C CNN
-F 1 "SW_SPDT" H 6800 3644 50  0000 C CNN
-F 2 "" H 6800 3450 50  0001 C CNN
-F 3 "" H 6800 3450 50  0001 C CNN
-	1    6800 3450
-	1    0    0    -1
-$EndComp
-Wire Wire Line
-	7000 3550 7000 3850
-Wire Wire Line
-	8300 3750 8300 3850
-Wire Wire Line
-	8300 3850 7000 3850
-Connection ~ 8300 3850
-Wire Wire Line
-	8300 3850 8300 4000
+	5150 3750 5250 3750
 Connection ~ 5350 3450
 Connection ~ 5350 3750
@@
 Connection ~ 5700 3450
 Connection ~ 5700 3750
-Wire Wire Line
-	5700 3450 6050 3450
-Wire Wire Line
-	5700 3750 6050 3750
-Connection ~ 6050 3450
-Connection ~ 6050 3750
-Wire Wire Line
-	6050 3450 6400 3450
-Wire Wire Line
-	6050 3750 6400 3750
-Connection ~ 6400 3450
-Connection ~ 6400 3750
-Wire Wire Line
-	6400 3450 6600 3450
-Wire Wire Line
-	6400 3750 6750 3750
-Connection ~ 7150 3750
-Wire Wire Line
-	7000 3350 7150 3350
-Wire Wire Line
-	7150 3450 7150 3350
-Wire Wire Line
-	7250 3350 7150 3350
-Connection ~ 7150 3350
-Wire Wire Line
-	7150 3750 7550 3750
-Wire Wire Line
-	7550 3650 7550 3750
-Connection ~ 7550 3750
-Wire Wire Line
-	7550 3750 7950 3750
-Wire Wire Line
-	7850 3350 7950 3350
-Wire Wire Line
-	8300 3350 8300 3450
-Wire Wire Line
-	7950 3450 7950 3350
-Connection ~ 7950 3350
-Wire Wire Line
-	7950 3350 8300 3350
-Wire Wire Line
-	7950 3750 8200 3750
-Wire Wire Line
-	8200 3750 8200 4000
-Connection ~ 7950 3750
 $Comp
 L Connector:Conn_01x01_Female SHIELD1
@@
 F 0 "SHIELD1" V 4447 4448 50  0000 L CNN
 F 1 "Conn_01x01_Female" V 4538 4448 50  0000 L CNN
-F 2 "" H 4600 4400 50  0001 C CNN
+F 2 "Connector_Wire:SolderWirePad_1x01_Drill1mm" H 4600 4400 50  0001 C CNN
 F 3 "~" H 4600 4400 50  0001 C CNN
 	1    4600 4400
@@
 L power:GND #PWR01
 U 1 1 5B6343B3
-P 6750 3950
-F 0 "#PWR01" H 6750 3700 50  0001 C CNN
-F 1 "GND" H 6755 3777 50  0000 C CNN
-F 2 "" H 6750 3950 50  0001 C CNN
-F 3 "" H 6750 3950 50  0001 C CNN
-	1    6750 3950
-	1    0    0    -1
-$EndComp
-Wire Wire Line
-	6750 3950 6750 3750
+P 5250 3850
+F 0 "#PWR01" H 5250 3600 50  0001 C CNN
+F 1 "GND" H 5255 3677 50  0000 C CNN
+F 2 "" H 5250 3850 50  0001 C CNN
+F 3 "" H 5250 3850 50  0001 C CNN
+	1    5250 3850
+	1    0    0    -1
+$EndComp
+Wire Wire Line
+	7650 3750 7650 3800
+Wire Wire Line
+	7550 3750 7650 3750
+Wire Wire Line
+	7750 3450 7750 3800
+Wire Wire Line
+	7550 3450 7750 3450
+Wire Wire Line
+	6850 3450 6750 3450
+Wire Wire Line
+	5250 3850 5250 3750
+Connection ~ 5250 3750
+Wire Wire Line
+	5250 3750 5350 3750
+Connection ~ 7550 3450
+Connection ~ 7550 3750
+Wire Wire Line
+	7150 3750 7550 3750
+Wire Wire Line
+	7450 3450 7550 3450
+Connection ~ 7150 3750
+Wire Wire Line
+	6750 3750 7150 3750
+Connection ~ 6750 3450
 Connection ~ 6750 3750
 Wire Wire Line
-	6750 3750 7150 3750
-$Comp
-L Diode:1N4001 D2
-U 1 1 5B6264B3
-P 8300 3600
-F 0 "D2" V 8346 3521 50  0000 R CNN
-F 1 "1N4001" V 8255 3521 50  0000 R CNN
-F 2 "Diode_THT:D_DO-41_SOD81_P10.16mm_Horizontal" H 8300 3425 50  0001 C CNN
-F 3 "http://www.vishay.com/docs/88503/1n4001.pdf" H 8300 3600 50  0001 C CNN
-	1    8300 3600
-	0    -1   -1   0
-$EndComp
+	5700 3450 6050 3450
+Wire Wire Line
+	5700 3750 6050 3750
+$Comp
+L Device:C C2
+U 1 1 5C0465F8
+P 6050 3600
+F 0 "C2" H 6165 3646 50  0000 L CNN
+F 1 "1uF" H 6165 3555 50  0000 L CNN
+F 2 "Capacitor_SMD:C_0805_2012Metric_Pad1.15x1.40mm_HandSolder" H 6088 3450 50  0001 C CNN
+F 3 "~" H 6050 3600 50  0001 C CNN
+	1    6050 3600
+	1    0    0    -1
+$EndComp
+Connection ~ 6050 3450
+Connection ~ 6050 3750
+Wire Wire Line
+	6400 3450 6750 3450
+Wire Wire Line
+	6400 3750 6750 3750
+Connection ~ 6400 3450
+Connection ~ 6400 3750
+Wire Wire Line
+	6050 3450 6400 3450
+Wire Wire Line
+	6050 3750 6400 3750
 $EndSCHEMATC

Commit message: Two alternatives for the USB power filter
Parts:
- C1: value UCL1E100MCL -> 100u; footprint Capacitor_SMD:CP_Elec_4x5.8 -> Capacitor_THT:CP_Radial_D5.0mm_P2.50mm
- POWER_IN1: footprint Connector_Wire:SolderWirePad_1x02_P3.81mm_Drill1mm -> Connector_PinHeader_2.54mm:PinHeader_1x02_P2.54mm_Vertical
- SHIELD1: footprint Connector_Wire:SolderWirePad_1x01_Drill1mm -> Connector_Wire:SolderWirePad_1x01_Drill0.8mm
Changed lines of the file:
@@
 EESchema Schematic File Version 4
+LIBS:USB_Power_Filter-cache
 EELAYER 26 0
 EELAYER END
@@
 P 5700 3600
 F 0 "C1" H 5650 3250 50  0000 L CNN
-F 1 "UCL1E100MCL" H 5400 3350 50  0000 L CNN
-F 2 "Capacitor_SMD:CP_Elec_4x5.8" H 5738 3450 50  0001 C CNN
+F 1 "100u" H 5400 3350 50  0000 L CNN
+F 2 "Capacitor_THT:CP_Radial_D5.0mm_P2.50mm" H 5738 3450 50  0001 C CNN
 F 3 "~" H 5700 3600 50  0001 C CNN
 	1    5700 3600
@@
 F 0 "POWER_IN1" V 5400 3100 50  0000 C CNN
 F 1 "Conn_01x02_Female" V 5300 3100 50  0000 C CNN
-F 2 "Connector_Wire:SolderWirePad_1x02_P3.81mm_Drill1mm" H 5250 3100 50  0001 C CNN
+F 2 "Connector_PinHeader_2.54mm:PinHeader_1x02_P2.54mm_Vertical" H 5250 3100 50  0001 C CNN
 F 3 "~" H 5250 3100 50  0001 C CNN
 	1    5250 3100
@@
 F 0 "SHIELD1" V 4447 4448 50  0000 L CNN
 F 1 "Conn_01x01_Female" V 4538 4448 50  0000 L CNN
-F 2 "Connector_Wire:SolderWirePad_1x01_Drill1mm" H 4600 4400 50  0001 C CNN
+F 2 "Connector_Wire:SolderWirePad_1x01_Drill0.8mm" H 4600 4400 50  0001 C CNN
 F 3 "~" H 4600 4400 50  0001 C CNN
 	1    4600 4400

Commit message: As sent to fab
Parts:
- D1: footprint Diode_SMD:D_SMB_Handsoldering -> Diode_SMD:D_SOD-323_HandSoldering
Changed lines of the file:
@@
 P 5700 3600
 F 0 "C1" H 5650 3250 50  0000 L CNN
-F 1 "100u" H 5400 3350 50  0000 L CNN
+F 1 "100u" H 5650 3350 50  0000 L CNN
 F 2 "Capacitor_THT:CP_Radial_D5.0mm_P2.50mm" H 5738 3450 50  0001 C CNN
 F 3 "~" H 5700 3600 50  0001 C CNN
@@
 F 0 "D1" V 5304 3679 50  0000 L CNN
 F 1 "D_TVS" V 5395 3679 50  0000 L CNN
-F 2 "Diode_SMD:D_SMB_Handsoldering" H 5350 3600 50  0001 C CNN
+F 2 "Diode_SMD:D_SOD-323_HandSoldering" H 5350 3600 50  0001 C CNN
 F 3 "~" H 5350 3600 50  0001 C CNN
 	1    5350 3600
