File: AISFilterAmp/AISFilterAmp.kicad_pcb (KiCad board)
At the start: 2 copper layers, 40 x 39 mm, 26 parts, among them U1 MSA0505, U2 LM2731XMF

Commit message: AISFilterAmp
Parts:
- moved PWR_J1 1.55 mm to (122.1, 120.7)
Routing:
- net Net-(PWR_C1-Pad1): track 19.9 -> 22.2 mm
- net GND: vias 76 -> 80
Other:
- outline, holes or cut-outs redrawn
