File: LED_MCU/LED_MCU.kicad_pcb (KiCad board)
At the start: 2 copper layers, 60 x 35 mm, 57 parts, among them J1 Wuerth_629105150521, J2 JST_PH_BAT, J3 ADDL_LED, U1 ATSAMD21G16B-AU, U2 AP2112K-3.3, U3 LDL1117S33R, U4 MCP73831-2-OT, U5 MAX17055ETB

Commit message: LED_MCU
Parts:
- removed C10, C12, C6: 1uF, Capacitor_SMD:C_0805_2012Metric_Pad1.15x1.40mm_HandSolder
- removed C11, C5, C7, C9: 10uF, Capacitor_SMD:C_0805_2012Metric_Pad1.15x1.40mm_HandSolder
- removed C8: 470uF, Capacitor_THT:CP_Radial_D10.0mm_P5.00mm
- removed D1: D_USB, Diode_THT:D_DO-41_SOD81_P7.62mm_Horizontal
- removed D2: D_BAT, Diode_THT:D_DO-41_SOD81_P7.62mm_Horizontal
- removed D3: D_TVS, Diode_THT:D_DO-15_P10.16mm_Horizontal
- removed J3: ADDL_LED, Connector_PinHeader_1.27mm:PinHeader_2x04_P1.27mm_Vertical
- removed J_ANA1: Conn_01x04, Connector_PinHeader_1.27mm:PinHeader_1x05_P1.27mm_Vertical
- removed LED_W4: LED_W, Diode_SMD:D_1206_3216Metric_Pad1.42x1.75mm_HandSolder
- removed Q_B1, Q_G1, Q_R1, Q_W1: PZT2222A, Package_TO_SOT_SMD:SOT-223-3_TabPin2
- removed R10, R11, R12, R15, R9: 6.8, Resistor_SMD:R_1206_3216Metric_Pad1.42x1.75mm_HandSolder
- removed R13, R14: 10, Resistor_SMD:R_1206_3216Metric_Pad1.42x1.75mm_HandSolder
- removed R4: 1k, Resistor_SMD:R_0805_2012Metric_Pad1.15x1.40mm_HandSolder
- removed R5, R6, R7, R8: 470, Resistor_SMD:R_1206_3216Metric_Pad1.42x1.75mm_HandSolder
- removed U2: AP2112K-3.3, Package_TO_SOT_SMD:SOT-23-5
- removed U3: LDL1117S33R, Package_TO_SOT_SMD:SOT-223-3_TabPin2
- removed U4: MCP73831-2-OT, Package_TO_SOT_SMD:SOT-23-5
- removed U5: MAX17055ETB, Maxim:Maxim_TDFN-10-1EP_2.5x2mm_P0.4mm_HandSoldering_ThermalVias
- added BAT_C1: 4.7u, Capacitor_SMD:C_0805_2012Metric, F.Cu at (129.2, 110.0)
- added BAT_C2: 4.7u, Capacitor_SMD:C_0805_2012Metric, F.Cu at (123.2, 110.0)
- added BAT_C3: 0.1u, Capacitor_SMD:C_0805_2012Metric, F.Cu at (145.2, 104.2)
- added BAT_R1: 5k, Resistor_SMD:R_0805_2012Metric, F.Cu at (128.4, 107.0)
- added BAT_R2: 1k, Resistor_SMD:R_0805_2012Metric, F.Cu at (125.2, 106.0)
- added BAT_U1: LTC2942-1, Package_DFN_QFN:DFN-6-1EP_3x2mm_P0.5mm_EP1.65x1.35mm, F.Cu at (140.0, 103.5)
- added BAT_U2: MCP73831-2-OT, Package_TO_SOT_SMD:SOT-23-5, F.Cu at (126.2, 110.0)
- added CONN_BAT1: CONN_BAT, Connector_JST:JST_PH_S2B-PH-K_1x02_P2.00mm_Horizontal, B.Cu at (117.2, 104.2)
- added CONN_USB1: USB, Connector_USB:USB_Micro-B_Wuerth_629105150521_CircularHoles, F.Cu at (137.8, 110.8)
- added HELLO_LED1: HELLO, Diode_SMD:D_0805_2012Metric_Castellated, F.Cu at (159.5, 120.0)
- added HELLO_R1: 6.8, Resistor_SMD:R_1206_3216Metric, F.Cu at (159.2, 118.0)
- added IN_C1: 100n, Capacitor_SMD:C_0805_2012Metric, F.Cu at (127.5, 116.2)
- added IN_C2: 100n, Capacitor_SMD:C_0805_2012Metric, F.Cu at (127.5, 118.2)
- added IN_C3: 100n, Capacitor_SMD:C_0805_2012Metric, F.Cu at (131.2, 116.2)
- added IN_J1: Conn_02x03_Odd_Even, Connector_PinSocket_1.27mm:PinSocket_2x03_P1.27mm_Vertical, F.Cu at (124.2, 116.4)
- added IN_R1: 1k, Resistor_SMD:R_0805_2012Metric, F.Cu at (127.5, 120.1)
- added IN_R2: 1k, Resistor_SMD:R_0805_2012Metric, F.Cu at (132.1, 123.2)
- added IN_R3: 1k, Resistor_SMD:R_0805_2012Metric, F.Cu at (128.2, 124.1)
- added PWR_C1: 100n, Capacitor_SMD:C_0805_2012Metric, F.Cu at (145.0, 110.5)
- added PWR_C2: 330uF, Capacitor_THT:CP_Radial_D6.3mm_P2.50mm, F.Cu at (151.8, 104.0)
- added PWR_C3: 1u, Capacitor_SMD:C_0805_2012Metric, F.Cu at (140.2, 88.2)
- added PWR_C4: 4.7u, Capacitor_SMD:C_0805_2012Metric, F.Cu at (151.2, 86.0)
- added PWR_C5: 1u, Capacitor_SMD:C_0805_2012Metric, F.Cu at (168.8, 119.2)
- added PWR_C6: 10u, Capacitor_SMD:C_0805_2012Metric, F.Cu at (169.0, 116.2)
- added PWR_C7: 1u, Capacitor_SMD:C_0805_2012Metric, F.Cu at (165.5, 116.2)
- added PWR_CONN1: Conn_01x02, Connector_PinHeader_1.27mm:PinHeader_1x02_P1.27mm_Vertical, F.Cu at (147.8, 111.2)
- added PWR_D1: D_Schottky, Diode_SMD:D_SOD-123F, F.Cu at (143.5, 107.5)
- added PWR_Q1: DMG2301L, Package_TO_SOT_SMD:SOT-23, F.Cu at (147.8, 107.0)
- added PWR_R1: 10k, Resistor_SMD:R_0805_2012Metric, F.Cu at (162.8, 119.2)
- added PWR_U1: TPD3E001DRLR, Package_TO_SOT_SMD:SOT-553, F.Cu at (142.2, 110.8)
- added PWR_U2: AP2112K-3.3, Package_TO_SOT_SMD:SOT-23-5, F.Cu at (165.8, 119.2)
- added PWR_U3: LD1117S33TR_SOT223, Package_TO_SOT_SMD:SOT-223-3_TabPin2, F.Cu at (145.8, 85.0)
- added Q1: Q_DUAL_NMOS, Package_SO:SO-8_3.9x4.9mm_P1.27mm, F.Cu at (168.0, 80.0)
- added Q2: Q_DUAL_NMOS, Package_SO:SO-8_3.9x4.9mm_P1.27mm, F.Cu at (168.0, 90.5)
- added Q3: Q_DUAL_NMOS, Package_SO:SO-8_3.9x4.9mm_P1.27mm, F.Cu at (168.0, 101.0)
- added RB1: 470, Resistor_SMD:R_1206_3216Metric, F.Cu at (158.0, 103.0)
- added RB2: 6.8, Resistor_SMD:R_1206_3216Metric, B.Cu at (161.8, 106.5)
- added REF**: MountingHole_2.1mm, MountingHole:MountingHole_2.1mm, B.Cu at (173.2, 87.5)
- added REF**: MountingHole_2.1mm, MountingHole:MountingHole_2.1mm, B.Cu at (145.5, 101.0)
- added REF**: MountingHole_2.1mm, MountingHole:MountingHole_2.1mm, B.Cu at (145.5, 92.0)
- added REF**: MountingHole_2.1mm, MountingHole:MountingHole_2.1mm, B.Cu at (136.5, 92.0)
- added REF**: MountingHole_2.1mm, MountingHole:MountingHole_2.1mm, B.Cu at (182.2, 87.5)
- added REF**: MountingHole_2.1mm, MountingHole:MountingHole_2.1mm, B.Cu at (182.2, 78.5)
- added REF**: MountingHole_2.1mm, MountingHole:MountingHole_2.1mm, B.Cu at (173.2, 78.5)
- added REF**: MountingHole_2.1mm, MountingHole:MountingHole_2.1mm, B.Cu at (173.2, 105.5)
- added REF**: MountingHole_2.1mm, MountingHole:MountingHole_2.1mm, B.Cu at (182.2, 105.5)
- added REF**: MountingHole_2.1mm, MountingHole:MountingHole_2.1mm, B.Cu at (182.2, 114.5)
- added REF**: MountingHole_2.1mm, MountingHole:MountingHole_2.1mm, B.Cu at (173.2, 114.5)
- added REF**: MountingHole_2.1mm, MountingHole:MountingHole_2.1mm, B.Cu at (136.5, 101.0)
- added RG1: 470, Resistor_SMD:R_1206_3216Metric, F.Cu at (158.0, 92.5)
- added RG2: 10, Resistor_SMD:R_1206_3216Metric, B.Cu at (161.8, 96.0)
- added RR1: 470, Resistor_SMD:R_1206_3216Metric, F.Cu at (159.0, 80.8)
- added RR2: 10, Resistor_SMD:R_1206_3216Metric, B.Cu at (158.0, 85.5)
- added RW1: 470, Resistor_SMD:R_1206_3216Metric, F.Cu at (161.8, 78.2)
- added RW1-1: 6.8, Resistor_SMD:R_1206_3216Metric, F.Cu at (143.5, 96.2)
- added RW1-2: 6.8, Resistor_SMD:R_1206_3216Metric, F.Cu at (176.0, 84.8)
- added RW1-3: 6.8, Resistor_SMD:R_1206_3216Metric, F.Cu at (176.0, 108.2)
- added RW2: 470, Resistor_SMD:R_1206_3216Metric, F.Cu at (161.8, 89.0)
- added RW2-1: 6.8, Resistor_SMD:R_1206_3216Metric, F.Cu at (176.0, 91.0)
- added RW2-2: 6.8, Resistor_SMD:R_1206_3216Metric, F.Cu at (177.8, 88.8)
- added RW2-3: 6.8, Resistor_SMD:R_1206_3216Metric, F.Cu at (180.2, 94.0)
- added RW3: 470, Resistor_SMD:R_1206_3216Metric, F.Cu at (161.8, 99.5)
- added RW3-1: 6.8, Resistor_SMD:R_1206_3216Metric, F.Cu at (180.2, 98.8)
- added RW3-2: 6.8, Resistor_SMD:R_1206_3216Metric, F.Cu at (177.8, 104.2)
- added RW3-3: 6.8, Resistor_SMD:R_1206_3216Metric, F.Cu at (176.0, 102.0)
- C1: value 100nF -> 100n; footprint Capacitor_SMD:C_0805_2012Metric_Pad1.15x1.40mm_HandSolder -> Capacitor_SMD:C_0805_2012Metric; moved to F.Cu
- C2: value 1uF -> 1u; footprint Capacitor_SMD:C_0805_2012Metric_Pad1.15x1.40mm_HandSolder -> Capacitor_SMD:C_0805_2012Metric
- C3: value 0.1uF -> 100n; footprint Capacitor_SMD:C_0805_2012Metric_Pad1.15x1.40mm_HandSolder -> Capacitor_SMD:C_0805_2012Metric
- C4: value 4.7uF -> 100n; footprint Capacitor_SMD:C_0805_2012Metric_Pad1.15x1.40mm_HandSolder -> Capacitor_SMD:C_0805_2012Metric
- H2: value MountingHole -> MountingHole_Pad; footprint MountingHole:MountingHole_2.5mm -> MountingHole:MountingHole_2.7mm_M2.5_DIN965_Pad
- H3: value MountingHole_Pad -> MountingHole; footprint MountingHole:MountingHole_2.7mm_M2.5_DIN965_Pad -> MountingHole:MountingHole_2.5mm
- J1: value Wuerth_629105150521 -> Conn_02x05_Odd_Even; footprint Connector_USB:USB_Micro-B_Wuerth_629105150521_CircularHoles -> Connector_PinHeader_1.27mm:PinHeader_2x05_P1.27mm_Vertical
- J2: value JST_PH_BAT -> Conn_02x06_Row_Letter_Last; footprint Connector_JST:JST_PH_S2B-PH-SM4-TB_1x02-1MP_P2.00mm_Horizontal -> Connector_PinHeader_1.27mm:PinHeader_2x06_P1.27mm_Vertical
- LED_O1: value LED_CHG -> LED_O
- R1: value 5k -> 1k; footprint Resistor_SMD:R_0805_2012Metric_Pad1.15x1.40mm_HandSolder -> Resistor_SMD:R_0805_2012Metric
- R2: value 10k -> 4.7k; footprint Resistor_SMD:R_0805_2012Metric_Pad1.15x1.40mm_HandSolder -> Resistor_SMD:R_0805_2012Metric
- R3: value 10m -> 4.7k; footprint Resistor_SMD:R_0805_2012Metric_Pad1.15x1.40mm_HandSolder -> Resistor_SMD:R_0805_2012Metric
- U1: value ATSAMD21G16B-AU -> ATSAML21E16B-AUT; footprint Package_QFP:TQFP-48_7x7mm_P0.5mm -> Package_QFP:TQFP-32_7x7mm_P0.8mm
- moved H3 97.3 mm to (181.2, 74.2)
- moved LED_W2 70.9 mm to (177.8, 83.0), turned to 315 degrees
- moved J2 66.6 mm to (176.2, 93.2)
- moved J1 65.4 mm to (168.5, 108.0), turned to 0 degrees
- moved J_RESET1 65.4 mm to (160.0, 124.2), turned to 270 degrees
- moved H2 61.5 mm to (136.5, 74.0)
- moved C4 45.2 mm to (164.2, 109.6), turned to 180 degrees
- moved LED_W1 43.7 mm to (141.0, 96.2), turned to 270 degrees
- moved C3 43.2 mm to (165.2, 112.6)
- moved LED_R1 38.2 mm to (163.0, 85.5), turned to 180 degrees
- moved R1 37.8 mm to (169.2, 105.7), turned to 0 degrees
- moved H4 37.1 mm to (136.5, 119.0)
- moved C2 36.4 mm to (163.2, 112.6), turned to 270 degrees
- moved R3 33.4 mm to (151.6, 124.1), turned to 90 degrees
- moved J_I2C1 29.8 mm to (151.8, 118.2), turned to 90 degrees
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Connections:
- net /ADDL_W renamed Net-(LED_W1-Pad1)
- C1 pad 1: /V_BUS -> /VDD
- C2 pad 1: /V_BUS -> GND
- C2 pad 2: GND -> Net-(C2-Pad2)
- C3 pad 1: /V_BAT -> GND
- C3 pad 2: GND -> Net-(C2-Pad2)
- C4 pad 2: Net-(C4-Pad2) -> /VDD
- J1 pad 1: /V_USB -> /VDD
- J1 pad 2: /D- -> /SWIO
- J1 pad 3: /D+ -> GND
- J1 pad 4: (no net) -> /SWCLK
- J1 pad 6: Net-(J1-Pad6) -> (no net)
- J2 pad 1: /GND_BAT -> Net-(J2-Pad1)
- J2 pad 2: /V_BAT -> Net-(J2-Pad2)
- J_I2C1 pad 1: /SCL -> /SDA
- J_I2C1 pad 2: /SDA -> /SCL
- LED_O1 pad 2: /V_BUS -> /VBUS
- R1 pad 1: Net-(R1-Pad1) -> /VDD
- R1 pad 2: GND -> /SWCLK
- R2 pad 1: Net-(R2-Pad1) -> /VDD
- R2 pad 2: /V_BUS -> /SDA
- R3 pad 1: GND -> /VDD
- R3 pad 2: /GND_BAT -> /SCL
- U1 pad 1: /A0 -> (no net)
- U1 pad 10: /LED_G -> GND
- U1 pad 11: /LED_B -> /IN1
- U1 pad 12: /LED_W -> /IN2
- U1 pad 13: (no net) -> /IN3
- U1 pad 17: /VDD -> /SDA
- U1 pad 18: GND -> /SCL
- U1 pad 2: /A1 -> (no net)
- U1 pad 21: (no net) -> /HELLO
- U1 pad 22: (no net) -> /PWR_CC
- U1 pad 23: (no net) -> /D-
- U1 pad 24: (no net) -> /D+
- U1 pad 26: (no net) -> /RESET
- U1 pad 27: (no net) -> Net-(C2-Pad2)
- U1 pad 28: (no net) -> GND
- U1 pad 3: (no net) -> /LED_B
- U1 pad 30: (no net) -> /VDD
- U1 pad 31: /SDA -> /SWCLK
- U1 pad 32: /SCL -> /SWIO
- U1 pad 4: /AREF -> /LED_W3
- U1 pad 5: GND -> /LED_G
- U1 pad 6: /VDD -> /LED_W2
- U1 pad 7: (no net) -> /LED_R
- U1 pad 8: (no net) -> /LED_W1
- U1 pad 9: /LED_R -> /VDD
Routing:
- net /V_LED: track 122.5 -> 0.00 mm, vias 2 -> 0
- net Net-(LED_W1-Pad1): track 88.2 -> 6.67 mm, vias 2 -> 0
- net /V_BUS: track 72.0 -> 0.00 mm
- net /VDD: track 42.4 -> 3.19 mm
- net /LED_W1: track 0.00 -> 34.2 mm
- net /V_BAT: track 31.9 -> 0.00 mm, vias 1 -> 0
- net /LED_W2: track 0.00 -> 22.4 mm
- net /D+: track 20.2 -> 5.54 mm, vias 0 -> 2
- net /SDA: track 14.2 -> 0.00 mm, vias 1 -> 0
- net /D-: track 20.2 -> 6.23 mm, vias 0 -> 2
- net Net-(J2-Pad1): track 0.00 -> 11.4 mm
- net Net-(J2-Pad11): track 0.00 -> 11.3 mm
- net /SCL: track 10.9 -> 0.00 mm, vias 1 -> 0
- net /LED_W3: track 0.00 -> 10.8 mm
- net /VBUS: track 0.00 -> 10.1 mm
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- added copper zone on F.Cu, net (none)
- removed copper zone on B.Cu, net GND
- removed copper zone on F.Cu, net GND
Other:
- board size 60 x 35 mm -> 50 x 50 mm
- net class /V_BUS removed
- net class C4P2 removed
- net class D+ added: clearance 0.2, trace_width 0.2, via_dia 0.8, via_drill 0.4
- net class Default: trace_width 0.25 -> 0.45
- rule pad_to_mask_clearance: 0.051 -> 0
