File: Freq_Gen_MCU/Freq_Gen_MCU_M0.kicad_pcb (KiCad board)
At the start: 2 copper layers, 79.8 x 38.8 mm, 54 parts, among them U1 ATSAML21E15B-AUT

Commit message: Freq gen
Parts:
- moved LO_C1 3.68 mm to (161.7, 130.7), turned to 270 degrees
- moved CLK_Y1 3.31 mm to (151.3, 126.2)
- moved CLK_C1 3.18 mm to (157.1, 126.8)
- moved CLK_U1 3.18 mm to (157.6, 129.8)
- moved CLK_C2 3.18 mm to (158.2, 132.6)
- moved LO_C2 2.68 mm to (163.8, 124.8)
- moved LO_L1 2.57 mm to (162.8, 127.8)
- moved LO_C3 1.87 mm to (167.8, 127.8)
- moved LO_L2 1.37 mm to (165.8, 127.8), turned to 270 degrees
- moved LO_CONN1 1.20 mm to (176.2, 126.0)
- moved LO_C4 1.10 mm to (170.6, 124.2), turned to 135 degrees
- moved LO_L3 1.00 mm to (170.6, 127.8), turned to 45 degrees
Routing:
- net /GPIO1: track 0.00 -> 6.93 mm
- net /VDD: track 106.5 -> 109.5 mm
- net /SCL: track 31.1 -> 34.1 mm
- net /SDA: track 31.4 -> 34.4 mm
- net /CLK: track 5.68 -> 3.68 mm
- net Net-(LO_C3-Pad1): track 3.62 -> 4.15 mm
- net GND: vias 131 -> 130
Other:
- outline, holes or cut-outs redrawn
